File: Design/FC/flight_controller.kicad_sch (KiCad schematic)
At the start: 28 parts, among them U1 STM32H747BIT6, U3 BMI323, U4 MMC5983MA, U5 BMP390

Commit message: refactored pins
Connections:
- net TIM_8_CH_2 is gone; now on net R_SERVO_2_SIGNAL: R_Servo_2.3 (Pin_3), U1.205 (PI6)
- net EXT_DEV_INT_BARO: no longer U5.7 (INT)
- net GND: no longer L_Servo_4.1 (Pin_1), U5.3 (VSS)
- net TIM_4_CH_1: no longer R_Motor.2 (Pin_2)
- net R_SERVO_2_SIGNAL: now reaches U1.143 (PC7)
- net BARO_SPI_NSS: now reaches U1.25 (PF3)
- net BARO_SPI_NSS: now also U5.6 (CSB)
- net BARO_INT_1: now reaches U1.26 (PF4)
- net BARO_INT_1: now also U5.7 (INT)
- net BARO_SPI_SCK: now reaches U1.31 (PF7)
- net BARO_SPI_SCK: now also U4.1 (SCL/SPI_SCK), U5.2 (SCK)
- net BARO_SPI_MISO: now reaches U1.32 (PF8)
- net BARO_SPI_MISO: now also U4.16 (SDA/SPI_SDI), U4.5 (SPI_SDO), U5.5 (SDO)
- net BARO_SPI_MOSI: now reaches U1.33 (PF9)
- net BARO_SPI_MOSI: now also U5.4 (SDI)
- net MAG_SPI_NSS: now reaches U1.34 (PF10)
- net MAG_SPI_NSS: now also U4.4 (SPI_CS)
- net EXT_DEV_INT_IMU: no longer names the net of U1.64 (PB1)
- net EXT_DEV_INT_IMU: no longer U3.4 (INT1)
- net EXT_DEV_INT_MAG: no longer names the net of U1.65 (PB2)
- net EXT_DEV_INT_MAG: no longer U4.15 (INT)
- net I2C_2_SCL renamed GPS_SCL
- net I2C_2_SDA renamed GPS_SDA
- net SPI_1_MISO renamed IMU_SPI_MISO
- net IMU_SPI_MISO: no longer U4.5 (SPI_SDO), U5.5 (SDO)
- net SPI_1_MOSI renamed IMU_SPI_MOSI
- net IMU_SPI_MOSI: no longer U4.16 (SDA/SPI_SDI), U5.4 (SDI)
- net SPI_1_NSS_BARO: no longer names the net of U1.63 (PB0)
- net SPI_1_NSS_BARO: no longer U5.6 (CSB)
- net SPI_1_NSS_IMU renamed IMU_SPI_NSS
- net SPI_1_NSS_MAG renamed EXT_5_DEV_IMU
- net EXT_5_DEV_IMU: now also U3.4 (INT1); no longer U4.4 (SPI_CS)
- net SPI_1_SCK renamed IMU_SPI_SCK
- net IMU_SPI_SCK: no longer U4.1 (SCL/SPI_SCK), U5.2 (SCK)
- net TIM_12_CH_1 renamed L_MOTOR_1_SIGNAL
- net L_MOTOR_1_SIGNAL: now also L_Motor.2 (Pin_2)
- net TIM_12_CH_2 renamed R_MOTOR_1_SIGNAL
- net R_MOTOR_1_SIGNAL: now also R_Motor.2 (Pin_2)
- net TIM_16_CH_1 renamed EXT_6_DEV_INT_MAG
- net EXT_6_DEV_INT_MAG: now also U4.15 (INT); no longer L_Motor.2 (Pin_2)
- net TIM_5_CH_1 renamed L_SERVO_1_SIGNAL
- net TIM_5_CH_2 renamed L_SERVO_2_SIGNAL
- net TIM_5_CH_3 renamed L_SERVO_3_SIGNAL
- net TIM_5_CH_4 renamed L_SERVO_4_SIGNAL
- net TIM_8_CH_1 renamed R_SERVO_1_SIGNAL
- net TIM_8_CH_3 renamed R_SERVO_3_SIGNAL
- net TIM_8_CH_4 renamed R_SERVO_4_SIGNAL
- net USART_1_RX renamed DEBUG_RX
- net USART_1_TX renamed DEBUG_TX
- net USART_3_RX renamed GPS_RX
- net USART_3_TX renamed GPS_TX
Other:
- moved on the sheet: C47, JL_Servo_2, L_Motor, L_Servo_4, R_Motor, R_Servo_2, R_Servo_4, U1A, U1B, U1C

Commit message: add rf receiver connector
Parts:
- added RF_RECV_CONN: Conn_01x04, symbol Connector_Generic:Conn_01x04
Connections:
- net +5V: now also RF_RECV_CONN.3 (Pin_3)
- net BARO_SPI_MISO: no longer U4.16 (SDA/SPI_SDI)
- net BARO_SPI_MOSI: now also U4.16 (SDA/SPI_SDI)
- net GND: now also RF_RECV_CONN.4 (Pin_4)
- net RF_RECV_TX: now reaches U1.175 (PD5)
- net RF_RECV_TX: now also RF_RECV_CONN.1 (Pin_1)
- net RF_RECV_RX: now reaches U1.176 (PD6)
- net RF_RECV_RX: now also RF_RECV_CONN.2 (Pin_2)
Other:
- note added: "??????"
- note added: "Compass"
- note added: "Connections"
- note added: "Debug"
- note added: "GPS"
- note added: "IMU"
- note added: "Motors"
- note added: "RF Receiver"
- note added: "RF Receiver Connection"
- note added: "SX1280 (Rx SPI)"
- note added: "Servos"
