File: Design/FC/flight_controller.kicad_sch (KiCad schematic)
At the start: 43 parts, among them U1 STM32H747BIT6

Commit message: modified bom for serial connector
Parts:
- LM1, LS1, LS2, LS3, LS4, RM1, RS1, RS2, RS3, RS4, Serial1: PACKAGE_TYPE TH 2.5mm -> TH 2.50mm
Changed lines of the file:
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@@
 			)
 		)
-		(property "PACKAGE_TYPE" "TH 2.5mm"
+		(property "PACKAGE_TYPE" "TH 2.50mm"
 			(at 171.45 184.15 90)
 			(effects
@@
 			)
 		)
-		(property "PACKAGE_TYPE" "TH 2.5mm"
+		(property "PACKAGE_TYPE" "TH 2.50mm"
 			(at 195.58 184.15 90)
 			(effects
@@
 			)
 		)
-		(property "PACKAGE_TYPE" "TH 2.5mm"
+		(property "PACKAGE_TYPE" "TH 2.50mm"
 			(at 259.08 184.15 90)
 			(effects
@@
 			)
 		)
-		(property "PACKAGE_TYPE" "TH 2.5mm"
+		(property "PACKAGE_TYPE" "TH 2.50mm"
 			(at 180.34 238.76 90)
 			(effects
@@
 			)
 		)
-		(property "PACKAGE_TYPE" "TH 2.5mm"
+		(property "PACKAGE_TYPE" "TH 2.50mm"
 			(at 195.58 212.09 90)
 			(effects
@@
 			)
 		)
-		(property "PACKAGE_TYPE" "TH 2.5mm"
+		(property "PACKAGE_TYPE" "TH 2.50mm"
 			(at 172.72 81.28 90)
 			(effects
@@
 			)
 		)
-		(property "PACKAGE_TYPE" "TH 2.5mm"
+		(property "PACKAGE_TYPE" "TH 2.50mm"
 			(at 234.95 184.15 90)
 			(effects
@@
 			)
 		)
-		(property "PACKAGE_TYPE" "TH 2.5mm"
+		(property "PACKAGE_TYPE" "TH 2.50mm"
 			(at 233.68 214.63 90)
 			(effects
@@
 			)
 		)
-		(property "PACKAGE_TYPE" "TH 2.5mm"
+		(property "PACKAGE_TYPE" "TH 2.50mm"
 			(at 257.81 214.63 90)
 			(effects
@@
 			)
 		)
-		(property "PACKAGE_TYPE" "TH 2.5mm"
+		(property "PACKAGE_TYPE" "TH 2.50mm"
 			(at 171.45 212.09 90)
 			(effects
@@
 			)
 		)
-		(property "PACKAGE_TYPE" "TH 2.5mm"
+		(property "PACKAGE_TYPE" "TH 2.50mm"
 			(at 241.3 238.76 90)
 			(effects
