File: Design/V2/power.kicad_sch (KiCad schematic)
At the start: 46 parts, among them U1 STM32H747BIT6

Commit message: power board
Parts:
- added J1: MCU Power, Connector_PinHeader_2.54mm:PinHeader_2x03_P2.54mm_Vertical, symbol Connector_Generic:Conn_02x03_Odd_Even
- added J2: Left Side Servo Power, Connector_PinHeader_2.54mm:PinHeader_2x04_P2.54mm_Vertical, symbol Connector_Generic:Conn_02x04_Odd_Even
- added J3: Right Side Servo Power, Connector_PinHeader_2.54mm:PinHeader_2x04_P2.54mm_Vertical, symbol Connector_Generic:Conn_02x04_Odd_Even
- renumbered REG_2 to U6
Connections:
- net +5V: now also J1.1 (Pin_1), J1.3 (Pin_3), J1.5 (Pin_5)
- net GND: now also J1.2 (Pin_2), J1.4 (Pin_4), J1.6 (Pin_6), J2.2 (Pin_2), J2.4 (Pin_4), J2.6 (Pin_6), J2.8 (Pin_8), J3.2 (Pin_2), J3.4 (Pin_4), J3.6 (Pin_6), J3.8 (Pin_8)
- new net SERVO_VCC_1_2: J2.1 (Pin_1), J2.3 (Pin_3)
- new net SERVO_VCC_3_4: J2.5 (Pin_5), J2.7 (Pin_7)
- new net SERVO_VCC_5_6: J3.1 (Pin_1), J3.3 (Pin_3)
- new net SERVO_VCC_7_8: J3.5 (Pin_5), J3.7 (Pin_7)
Other:
- moved on the sheet: C10, C12, H1, H2, H3, H4, LED8, R3, U6

Commit message: editing bom
Parts:
- C10, C12: LCSC Part # (none) -> C19702; Manufacturer_Name Murata Electronics -> Samsung Electro-Mechanics; Manufacturer_Part_Number GRM188R61E106KA73D -> CL10A106KP8NNNC
- C11, C31: LCSC Part # (none) -> C19666; Manufacturer_Name Murata Electronics -> Samsung Electro-Mechanics; Manufacturer_Part_Number GRM188R61E475KE11D -> CL10A475KO8NNNC
- C13, C38: LCSC Part # (none) -> C2907032; Manufacturer_Name Murata Electronics -> Samsung Electro-Mechanics; Manufacturer_Part_Number GRM188R61A105KA61D -> CL10A105KB8NNNC
- C14, C15, C16, C17, C18, C19, C20, C21, C22, C23, C24, C25, C26, C27, C28, C29, C30, C32, C36, C37, C39, C40: LCSC Part # (none) -> C14663
- C34, C35, C41: LCSC Part # (none) -> C23630; Manufacturer_Name Taiyo Yuden -> Samsung Electro-Mechanics; Manufacturer_Part_Number TMK107ABJ225KA-T -> CL10A225KO8NNNC
- FB1: value FerriteBead_Small -> Ferrite Bead; LCSC Part # (none) -> C14709; Manufacturer_Name TDK Corporation -> Murata Electronics; Manufacturer_Part_Number MPZ1005S121HT000 -> BLM18PG121SN1D
- LED8: value G -> Red; LCSC Part # (none) -> C2286; Manufacturer_Name Lite-On Inc. -> Hubei KENTO Elec; Manufacturer_Part_Number LTW-C190DA5 -> KT-0603R
- R3: value 240 -> 39; LCSC Part # (none) -> C2907032; Manufacturer_Name Panasonic Electronic Components -> FOJAN; Manufacturer_Part_Number ERJ-PA3F5600V -> FRC0603F39R0TS
- U1: LCSC Part # (none) -> C730197
- U6: A_MAX 1.0 -> (none); B_MAX 0.45 -> (none); B_MIN 0.23 -> (none); B_NOM 0.34 -> (none); D2_NOM 2.365 -> (none); D_MAX 3.1 -> (none); D_MIN 2.9 -> (none); D_NOM 3.0 -> (none); E2_NOM 1.625 -> (none); ENOM 0.95 -> (none); E_MAX 3.1 -> (none); E_MIN 2.9 -> (none); E_NOM 3.0 -> (none); LCSC Part # (none) -> C222192; L_MAX 0.5 -> (none); L_MIN 0.3 -> (none); L_NOM 0.4 -> (none); MANUFACTURER ST Microelectronics -> (none); MAXIMUM_PACKAGE_HEIGHT 1.0mm -> (none); PARTREV 3 -> (none); PIN_COUNT 6.0 -> (none); STANDARD IPC 7351B -> (none)
