File: Design/V2/fc.kicad_pcb (KiCad board)
At the start: 4 copper layers, 70.8 x 100 mm, 116 parts, among them J1 XT60PW-M, U1 STM32H747BIT6, U2 INA219AIDCNT

Commit message: power board
Parts:
- removed +3.3V, +5V, GND: TestPoint_Pad_1.0x1.0mm, TestPoint:TestPoint_Pad_1.0x1.0mm
- removed C1: 100nF, Capacitor_SMD:C_0603_1608Metric_Pad1.08x0.95mm_HandSolder
- removed C2, C3: 22uF, Capacitor_SMD:C_1210_3225Metric_Pad1.33x2.70mm_HandSolder
- removed C4, C51: 2.2uF, Capacitor_SMD:C_0805_2012Metric_Pad1.18x1.45mm_HandSolder
- removed C5, C6: 0.1uF, Capacitor_SMD:C_0805_2012Metric_Pad1.18x1.45mm_HandSolder
- removed C50, C7, C9: 100uF, Lib:CAP_6.3 X 7.7_PAN
- removed C8: 4.7nF, Capacitor_SMD:C_0805_2012Metric_Pad1.18x1.45mm_HandSolder
- removed D1: SD103AW-TP, Diode_SMD:Nexperia_CFP3_SOD-123W
- removed J1: XT60PW-M, Lib:XT60PW-M
- removed L1: 6.8uH, Lib:IND_SRP1265A-6R8M_BRN
- removed LED1: G, LED_SMD:LED_0603_1608Metric
- removed R1: 0.01, Lib:RES_PE2512_YAG
- removed R2, R20: 10k, Lib:RES_ERJ-T06J103V_0805
- removed R4: 19.6k, Lib:RES_ERJ-PB6B1962V_0805
- removed R5: 6.8K, Resistor_SMD:R_0805_2012Metric_Pad1.20x1.40mm_HandSolder
- removed R6: 1.3K, Resistor_SMD:R_0805_2012Metric_Pad1.20x1.40mm_HandSolder
- removed R7: 560, Resistor_SMD:R_0603_1608Metric_Pad0.98x0.95mm_HandSolder
- removed REG_1: MIC26903YJL-TR, Lib:MIC26903YJL-TR-MLF28_5X6_MCH
- removed U2: INA219AIDCNT, Lib:INA219AIDCNT-SOT65P280X145-8N
- renumbered REG_2 to U6
Connections:
- C12 pad 1: +5V -> PWR_BRD_5V
- U6 pad 5: +5V -> PWR_BRD_5V
- U6 pad 6: +5V -> PWR_BRD_5V
Routing:
- net +5V: track 165.7 -> 9.17 mm, vias 43 -> 14
- net GND: track 243.1 -> 128.8 mm, vias 202 -> 141
- net CURRENT_SENSE_SCL: track 70.4 -> 7.26 mm, vias 2 -> 1
- net CURRENT_SENSE_SDA: track 70.1 -> 9.71 mm, vias 2 -> 1
- net +3.3V: track 266.0 -> 213.6 mm, vias 48 -> 47
- net REG_1_VIN: track 47.0 -> 0.00 mm
- net REG_1_CS: track 27.7 -> 0.00 mm, vias 2 -> 0
- net PWR_BRD_5V: track 0.00 -> 16.8 mm
- net REG_1_FB: track 15.6 -> 0.00 mm, vias 1 -> 0
- net /Power/REG_1_VDD: track 14.0 -> 0.00 mm, vias 1 -> 0
- net REG_1_PG: track 6.95 -> 0.00 mm, vias 1 -> 0
- net VIN+: track 6.40 -> 0.00 mm
- net REG_1_BST: track 5.65 -> 0.00 mm, vias 1 -> 0
- net REG_1_EN: track 5.61 -> 0.00 mm
- net /Power/REG_1_PVDD: track 5.28 -> 0.00 mm, vias 1 -> 0
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- removed copper zone on F.Cu, net REG_1_CS
- removed copper zone on F.Cu, net REG_1_VIN
- removed copper zone on F.Cu, net VIN+
Other:
- board size 70.8 x 100 mm -> 70.8 x 125 mm
- board text removed: "+"
- board text removed: "-"

Commit message: added test pads for gps rf and debug
Parts:
- removed GPS1: Conn_01x06, Molex:CONN_532610001-SD_06Pin_1.25mm
- removed RF1: Conn_01x04, Molex:CONN_532610471_SMD_4Pin_1.25mm
- removed Serial1: Conn_01x03, Connector_PinHeader_2.54mm:PinHeader_1x03_P2.54mm_Vertical
- added 5V: TestPoint, TestPoint:TestPoint_Pad_1.0x1.0mm, F.Cu at (217.0, 148.8)
- added 5V: TestPoint, TestPoint:TestPoint_Pad_1.0x1.0mm, F.Cu at (230.2, 93.5)
- added GND: TestPoint, TestPoint:TestPoint_Pad_1.0x1.0mm, F.Cu at (211.1, 148.8)
- added GND: TestPoint, TestPoint:TestPoint_Pad_1.0x1.0mm, F.Cu at (230.2, 99.7)
- added GND: TestPoint, TestPoint:TestPoint_Pad_1.0x1.0mm, F.Cu at (261.1, 131.5)
- added J1: MCU Power, Connector_PinHeader_2.54mm:PinHeader_2x03_P2.54mm_Vertical, F.Cu at (195.9, 88.1)
- added J2: Left Side Servo Power, Connector_PinHeader_2.54mm:PinHeader_2x04_P2.54mm_Vertical, F.Cu at (255.8, 111.9)
- added J3: Right Side Servo Power, Connector_PinHeader_2.54mm:PinHeader_2x04_P2.54mm_Vertical, F.Cu at (262.9, 111.9)
- added RX: TestPoint, TestPoint:TestPoint_Pad_1.0x1.0mm, F.Cu at (213.0, 148.8)
- added RX: TestPoint, TestPoint:TestPoint_Pad_1.0x1.0mm, F.Cu at (261.1, 128.4)
- added RX: TestPoint, TestPoint:TestPoint_Pad_1.0x1.0mm, F.Cu at (230.2, 97.6)
- added TX: TestPoint, TestPoint:TestPoint_Pad_1.0x1.0mm, F.Cu at (230.2, 95.5)
- added TX: TestPoint, TestPoint:TestPoint_Pad_1.0x1.0mm, F.Cu at (215.0, 148.8)
- added TX: TestPoint, TestPoint:TestPoint_Pad_1.0x1.0mm, F.Cu at (261.1, 125.4)
- FB1: value FerriteBead_Small -> Ferrite Bead
- LED3, LED7: value R -> Red
- LED4: value Y -> Red
- LED5, LED6: value B -> Red
- LED8: value G -> Red
- R15, R16, R17, R18, R19: value 330 -> 39
- R3: value 240 -> 39
Connections:
- C12 pad 1: PWR_BRD_5V -> +5V
- U6 pad 5: PWR_BRD_5V -> +5V
- U6 pad 6: PWR_BRD_5V -> +5V
Routing:
- net DEBUG_RX: track 19.5 -> 0.00 mm
- net DEBUG_TX: track 18.6 -> 0.00 mm
- net PWR_BRD_5V: track 16.8 -> 0.00 mm
- net GND: track 128.8 -> 120.7 mm, vias 141 -> 137
- net +5V: track 9.17 -> 16.8 mm, vias 14 -> 10
- net RF_RECV_RX: track 31.6 -> 25.6 mm
- net RF_RECV_TX: track 29.7 -> 24.9 mm
- net GPS_TX: track 19.8 -> 18.0 mm
Other:
- board size 70.8 x 125 mm -> 70.8 x 100 mm
- board text added: "DB"
- board text added: "RF"
- board text removed: "+5V"
- board text removed: "TX"
