File: Design/V2/power_brd/power_brd.kicad_sch (KiCad schematic)
At the start: 58 parts, among them J1 XT60PW-M, J2 Conn_02x03_Odd_Even, J3 Conn_02x04_Odd_Even, J4 Conn_02x04_Odd_Even, U1 TPS5430DDAR, U2 TPS5430DDAR, U3 TPS5430DDAR, U4 TPS5430DDAR, U5 TPS5430DDAR

Commit message: fc and power board sent out for assembly
Parts:
- C1, C13, C4, C7, C8: LCSC Part # (none) -> C13585; Manufacturer (none) -> Samsung Electro-Mechanics; Manufacturer ID (none) -> CL31A106KBHNNNE
- C10, C14, C3, C5, C9: LCSC Part # (none) -> C1710; Manufacturer (none) -> Samsung Electro-Mechanics; Manufacturer ID (none) -> CL21B103KBANNNC
- C11, C12, C15, C2, C6: LCSC Part # (none) -> C147767; Manufacturer (none) -> PANASONIC; Manufacturer ID (none) -> 10TPE220ML
- D1, D2, D3, D4, D5: footprint Diodes:SS34_DO214AB -> Diodes:SMA_L4.3-W2.6-LS5.2-RD; LCSC Part # (none) -> C8678; Manufacturer (none) -> MDD(Microdiode Semiconductor); Manufacturer ID (none) -> SS34
- D10, D6, D7, D8, D9: LCSC Part # (none) -> C84256; Manufacturer (none) -> Foshan NationStar Optoelectronics; Manufacturer ID (none) -> NCD0805R1
- J1: Availability Not in stock -> (none); Check_prices https://www.snapeda.com/parts/XT60PW-M/AMASS/view-part/?ref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 -> (none); Description_1 Socket, DC supply, male, PIN: 2 -> (none); MANUFACTURER AMASS -> (none); MAXIMUM_PACKAGE_HEIGHT 8.4 mm -> (none); MF AMASS -> (none); PARTREV V1.2 -> (none); Price None -> (none); STANDARD Manufacturer recommendations -> (none); SnapEDA_Link https://www.snapeda.com/parts/XT60PW-M/AMASS/view-part/?ref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 -> (none); now left out of the parts list
- J2, J3, J4: now left out of the parts list
- L1, L2, L3, L4, L5: LCSC Part # (none) -> C22463824; Manufacturer (none) -> TECHFUSE; Manufacturer ID (none) -> SL0630-150M
- R1, R3, R5, R7, R9: LCSC Part # (none) -> C17414; Manufacturer (none) -> UNI-ROYAL(Uniroyal Elec); Manufacturer ID (none) -> 0805W8F1002T5E
- R10, R2, R4, R6, R8: LCSC Part # (none) -> C17609; Manufacturer (none) -> UNI-ROYAL(Uniroyal Elec); Manufacturer ID (none) -> 0805W8F3241T5E
- R11, R12, R13, R14, R15: LCSC Part # (none) -> C17408; Manufacturer (none) -> UNI-ROYAL(Uniroyal Elec); Manufacturer ID (none) -> 0805W8F1000T5E
- U1, U2, U3, U4, U5: LCSC Part # (none) -> C9864; Manufacturer (none) -> Texas Instruments; Manufacturer ID (none) -> TPS5430DDAR
